Commit message: Update arm.xacro
add inertial to the base

File: arm20/urdf/arm.xacro (robot description, xacro)
@@ -108,4 +108,9 @@
   </joint>
   <link name="base_link">
+       <inertial>
+            <origin xyz="${origin_base_xyz}" rpy="0.0 0.0 0.0"/>
+            <mass value="1.05"/>
+            <inertia ixx="1.01" ixy="0.0" ixz="0.0" iyy="1.01" iyz="0.0" izz="1.01"/>
+       </inertial>
        <visual>
           <origin xyz="${origin_base_xyz}" rpy="0.0 0.0 0.0"/>
